Commit message: diffential robot

File: description/gazebo_control.xacro (robot description, xacro)
@@ -19,5 +19,5 @@
             <!-- OUTPUTS-->
             <odometry_frame>odom</odometry_frame>
-            <robot_base_frame>base_link</robot_base_frame><!-- standard link-->
+            <robot_base_frame>base_footprint</robot_base_frame><!-- standard link-->
             <publish_odom>true</publish_odom><!-- publish odom if had message "true"-->
             <publish_odom_tf>true</publish_odom_tf>

File: description/robot.urdf.xacro (robot description, xacro)
@@ -1,5 +1,6 @@
 <?xml version="1.0"?>
 <robot xmlns:xacro="http://www.ros.org/wiki/xacro" name="robot">
-    <xacro:include filename="robot_core.xacro" />
+    <xacro:include filename="robot_core_differential_robot.xacro" />
+    <!-- <xacro:include filename="robot_core_four_wheel_.xacro" /> -->
     <xacro:include filename="gazebo_control.xacro" />
 </robot>

File: description/robot_core_four_wheel_.xacro (robot description, xacro)
@@ -105,5 +105,5 @@
     <!--LEFT
     WHEEL FOWARD LINK-->
-    <joint name="left_wheel_foward_joint" type="continuous">
+    <joint name="left_wheel_foward_joint" type="fixed">
         <parent link="base_link" />
         <child link="left_wheel_foward_link" />
@@ -135,5 +135,5 @@
     <!--RIGHT
     WHEEL FOWARD LINK-->
-    <joint name="right_wheel_foward_joint" type="continuous">
+    <joint name="right_wheel_foward_joint" type="fixed">
         <parent link="base_link" />
         <child link="right_wheel_foward_link" />
