Commit message: add lidar2D xacro file

File: description/robot.urdf.xacro (robot description, xacro)
@@ -4,3 +4,4 @@
     <!-- <xacro:include filename="robot_core_four_wheel_.xacro" /> -->
     <xacro:include filename="gazebo_control.xacro" />
+    <xacro:include filename="lidar2D.xacro" />
 </robot>

File: description/robot_core_differential_robot.xacro (robot description, xacro)
@@ -13,4 +13,7 @@
     <material name="black">
         <color rgba="0 0 0 1" />
+    </material>
+    <material name="red">
+        <color rgba="1 0 0 1" />
     </material>
     <!--BASE
@@ -50,8 +53,8 @@
     WHEEL BACK LINK-->
     <joint name="left_wheel_back_joint" type="continuous">
-        <parent link="base_footprint" />
+        <parent link="base_link" />
         <child link="left_wheel_back_link" />
         <origin
-            xyz="-0.075 0.116 0.0625" rpy="-${pi/2} 0.0 0.0" /><!-- 116 = 90+52/2-->
+            xyz="-0.075 0.116 0.0" rpy="-${pi/2} 0.0 0.0" /><!-- 116 = 90+52/2-->
         <axis xyz="0.0 0.0 1" />
     </joint>
@@ -79,7 +82,7 @@
     WHEEL BACK LINK-->
     <joint name="right_wheel_back_joint" type="continuous">
-        <parent link="base_footprint" />
+        <parent link="base_link" />
         <child link="right_wheel_back_link" />
-        <origin xyz="-0.075 -0.116 0.0625" rpy="${pi/2} 0.0 0.0" /><!-- 116 = 90+52/2-->
+        <origin xyz="-0.075 -0.116 0.0" rpy="${pi/2} 0.0 0.0" /><!-- 116 = 90+52/2-->
         <axis xyz="0.0 0.0 -1" />
     </joint>
