Commit message: add <sphere radius=0.0625 /> in collision

File: description/robot_core_differential_robot.xacro (robot description, xacro)
@@ -68,5 +68,6 @@
         <collision>
             <geometry>
-                <cylinder radius="0.0625" length="0.05132" />
+                <!-- <cylinder radius="0.0625" length="0.05132" /> -->
+                <sphere radius="0.0625" />
             </geometry>
             <!-- <material name="orange" /> -->
@@ -96,5 +97,6 @@
         <collision>
             <geometry>
-                <cylinder radius="0.0625" length="0.05132" />
+                <!-- <cylinder radius="0.0625" length="0.05132" /> -->
+                <sphere radius="0.0625" />
             </geometry>
             <!-- <material name="orange" /> -->
