Commit message: create branch for Real robot

File: description/ros2_control.xacro (robot description, xacro)
@@ -1,4 +1,25 @@
 <?xml version="1.0"?>
 <robot xmlns:xacro="http://www.ros.org/wiki/xacro">
+    <!-- <ros2_control name="GazeboSystem" type="system">
+        <hardware>
+            <plugin>gazebo_ros2_control/GazeboSystem</plugin>
+        </hardware>
+        <joint name="left_wheel_back_joint">
+            <command_interface name="velocity">
+                <param name="min">-10</param>
+                <param name="max"> 10</param>
+            </command_interface>
+            <state_interface name="velocity" />
+            <state_interface name="position" />
+        </joint>
+        <joint name="right_wheel_back_joint">
+            <command_interface name="velocity">
+                <param name="min">-10</param>
+                <param name="max"> 10</param>
+            </command_interface>
+            <state_interface name="velocity" />
+            <state_interface name="position" />
+        </joint>
+    </ros2_control> -->
     <ros2_control name="GazeboSystem" type="system">
         <hardware>
